File: MB-C2.Auduino_Nano_R4/KiCad/MB-C2/MB-C2.kicad_sch (KiCad schematic)
At the start: 37 parts, among them J1 PH-2x15SG, J2 PH-2x15SG, J3 Cut_of_PH-2x40RG, J4 Barrel_Jack_Switch, J5 Conn_02x04_Odd_Even, J6 Servo 3x2 header, J7 Servo 3x2 header, J8 Conn_01x04_Pin, Q1 INK021ABS1-T112, Q2 INK021ABS1-T112, Q3 INK021ABS1-T112, Q4 INK021ABS1-T112, U1 AE-G5V-DRV, U2 AE-G5V-DRV, U3 AE-G5V-DRV, U4 AE-G5V-DRV

Commit message: [MB-C2:KiCAD] Change to double side PCB
- Change design rule to JLCPB capability.
- Remove jumper resisters.
- Migrate power lines to front side.
Parts:
- removed R1: 0, 01_Prj_Local_Footpint:R_Axial_DIN0204_L3.6mm_D1.6mm_P10.16mm_Horizontal_TMVC, symbol Device:R_US
- removed R10: 0, 01_Prj_Local_Footpint:R_Axial_DIN0204_L3.6mm_D1.6mm_P7.62mm_Horizontal_TMVC, symbol Device:R_US
- renumbered R2 to R1, R9 to R10, R3 to R2, R4 to R3, R5 to R4, R6 to R5, R7 to R6, R8 to R7, R11 to R8, R12 to R9
Connections:
- net +5VP: now also J3.13 (Pin_13), J3.14 (Pin_14)
- net PIN27_5V: now also D1.1 (K), D2.1 (K), D5.1 (K), D6.1 (K)
Changed lines of the file:
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@@
 	(wire
 		(pts
-			(xy 233.68 21.59) (xy 236.22 21.59)
-		)
-		(stroke
-			(width 0)
-			(type default)
-		)
-	)
-	(wire
-		(pts
 			(xy 15.24 101.6) (xy 34.29 101.6)
 		)
@@
 	(wire
 		(pts
-			(xy 34.29 102.87) (xy 34.29 101.6)
+			(xy 34.29 101.6) (xy 34.29 110.49)
 		)
 		(stroke
@@
 	(wire
 		(pts
-			(xy 246.38 21.59) (xy 246.38 19.05)
-		)
-		(stroke
-			(width 0)
-			(type default)
-		)
-	)
-	(wire
-		(pts
 			(xy 124.46 35.56) (xy 139.7 35.56)
 		)
@@
 		)
 	)
-	(wire
-		(pts
-			(xy 243.84 21.59) (xy 246.38 21.59)
-		)
-		(stroke
-			(width 0)
-			(type default)
-		)
-	)
 	(label "D6"
 		(at 63.5 43.18 0)
@@
 		(on_board yes)
 		(dnp no)
-		(property "Reference" "R2"
+		(property "Reference" "R1"
 			(at 121.666 113.03 90)
 			(effects
@@
 			(project "MB-C2"
 				(path "/da3163b4-b098-4cd4-9588-703f26f78e93"
-					(reference "R2")
+					(reference "R1")
 					(unit 1)
 				)
@@
 		(on_board yes)
 		(dnp no)
-		(property "Reference" "R3"
+		(property "Reference" "R2"
 			(at 37.338 118.11 90)
 			(effects
@@
 			(project ""
 				(path "/da3163b4-b098-4cd4-9588-703f26f78e93"
-					(reference "R3")
-					(unit 1)
-				)
-			)
-		)
-	)
-	(symbol
-		(lib_id "Device:R_US")
-		(at 240.03 21.59 90)
-		(unit 1)
-		(exclude_from_sim no)
-		(in_bom yes)
-		(on_board yes)
-		(dnp no)
-		(property "Reference" "R10"
-			(at 236.728 19.05 90)
-			(effects
-				(font
-					(size 1.27 1.27)
-				)
-			)
-		)
-		(property "Value" "0"
-			(at 241.3 23.622 90)
-			(effects
-				(font
-					(size 1.27 1.27)
-				)
-			)
-		)
-		(property "Footprint" "01_Prj_Local_Footpint:R_Axial_DIN0204_L3.6mm_D1.6mm_P7.62mm_Horizontal_TMVC"
-			(at 240.284 20.574 90)
-			(effects
-				(font
-					(size 1.27 1.27)
-				)
-				(hide yes)
-			)
-		)
-		(property "Datasheet" "~"
-			(at 240.03 21.59 0)
-			(effects
-				(font
-					(size 1.27 1.27)
-				)
-				(hide yes)
-			)
-		)
-		(property "Description" "Resistor, US symbol"
-			(at 240.03 21.59 0)
-			(effects
-				(font
-					(size 1.27 1.27)
-				)
-				(hide yes)
-			)
-		)
-		(pin "1"
-		)
-		(pin "2"
-		)
-		(instances
-			(project "MB-C2"
-				(path "/da3163b4-b098-4cd4-9588-703f26f78e93"
-					(reference "R10")
+					(reference "R2")
 					(unit 1)
 				)
@@
 		(dnp no)
 		(fields_autoplaced yes)
-		(property "Reference" "R11"
+		(property "Reference" "R8"
 			(at 41.91 176.5299 0)
 			(effects
@@
 			(project "MB-C2"
 				(path "/da3163b4-b098-4cd4-9588-703f26f78e93"
-					(reference "R11")
+					(reference "R8")
 					(unit 1)
 				)
@@
 		(on_board yes)
 		(dnp no)
-		(property "Reference" "R8"
+		(property "Reference" "R7"
 			(at 121.666 161.29 90)
 			(effects
@@
 			(project "MB-C2"
 				(path "/da3163b4-b098-4cd4-9588-703f26f78e93"
-					(reference "R8")
+					(reference "R7")
 					(unit 1)
 				)
@@
 		(on_board yes)
 		(dnp no)
-		(property "Reference" "R9"
+		(property "Reference" "R10"
 			(at 121.666 185.42 90)
 			(effects
@@
 			(project "MB-C2"
 				(path "/da3163b4-b098-4cd4-9588-703f26f78e93"
-					(reference "R9")
+					(reference "R10")
 					(unit 1)
 				)
@@
 		(dnp no)
 		(fields_autoplaced yes)
-		(property "Reference" "R12"
+		(property "Reference" "R9"
 			(at 50.8 176.5299 0)
 			(effects
@@
 			(project "MB-C2"
 				(path "/da3163b4-b098-4cd4-9588-703f26f78e93"
-					(reference "R12")
+					(reference "R9")
 					(unit 1)
 				)
@@
 		(on_board yes)
 		(dnp no)
-		(property "Reference" "R5"
+		(property "Reference" "R4"
 			(at 121.666 137.16 90)
 			(effects
@@
 			(project "MB-C2"
 				(path "/da3163b4-b098-4cd4-9588-703f26f78e93"
-					(reference "R5")
+					(reference "R4")
 					(unit 1)
 				)
@@
 		(on_board yes)
 		(dnp no)
-		(property "Reference" "R6"
+		(property "Reference" "R5"
 			(at 38.354 137.16 90)
 			(effects
@@
 			(project "MB-C2"
 				(path "/da3163b4-b098-4cd4-9588-703f26f78e93"
-					(reference "R6")
+					(reference "R5")
 					(unit 1)
 				)
@@
 	(symbol
 		(lib_id "power:+5VP")
-		(at 246.38 19.05 0)
+		(at 233.68 21.59 0)
 		(unit 1)
 		(exclude_from_sim no)
@@
 		(fields_autoplaced yes)
 		(property "Reference" "#PWR02"
-			(at 246.38 22.86 0)
+			(at 233.68 25.4 0)
 			(effects
 				(font
@@
 		)
 		(property "Value" "+5VP"
-			(at 246.38 13.97 0)
+			(at 233.68 16.51 0)
 			(effects
 				(font
@@
 		)
 		(property "Footprint" ""
-			(at 246.38 19.05 0)
+			(at 233.68 21.59 0)
 			(effects
 				(font
@@
 		)
 		(property "Datasheet" ""
-			(at 246.38 19.05 0)
+			(at 233.68 21.59 0)
 			(effects
 				(font
@@
 		)
 		(property "Description" "Power symbol creates a global label with name \"+5VP\""
-			(at 246.38 19.05 0)
+			(at 233.68 21.59 0)
 			(effects
 				(font
@@
 		(on_board yes)
 		(dnp no)
-		(property "Reference" "R7"
+		(property "Reference" "R6"
 			(at 72.898 137.16 90)
 			(effects
@@
 			(project "MB-C2"
 				(path "/da3163b4-b098-4cd4-9588-703f26f78e93"
-					(reference "R7")
+					(reference "R6")
 					(unit 1)
 				)
@@
 		(on_board yes)
 		(dnp no)
-		(property "Reference" "R4"
+		(property "Reference" "R3"
 			(at 72.644 118.618 90)
 			(effects
@@
 			(project "MB-C2"
 				(path "/da3163b4-b098-4cd4-9588-703f26f78e93"
-					(reference "R4")
+					(reference "R3")
 					(unit 1)
 				)
@@
 					(unit 1)
 				)
-			)
-		)
-	)
-	(symbol
-		(lib_id "Device:R_US")
-		(at 34.29 106.68 0)
-		(unit 1)
-		(exclude_from_sim no)
-		(in_bom yes)
-		(on_board yes)
-		(dnp no)
-		(fields_autoplaced yes)
-		(property "Reference" "R1"
-			(at 36.83 105.4099 0)
-			(effects
-				(font
-					(size 1.27 1.27)
-				)
-				(justify left)
-			)
-		)
-		(property "Value" "0"
-			(at 36.83 107.9499 0)
-			(effects
-				(font
-					(size 1.27 1.27)
-				)
-				(justify left)
-			)
-		)
-		(property "Footprint" "01_Prj_Local_Footpint:R_Axial_DIN0204_L3.6mm_D1.6mm_P10.16mm_Horizontal_TMVC"
-			(at 35.306 106.934 90)
-			(effects
-				(font
-					(size 1.27 1.27)
-				)
-				(hide yes)
-			)
-		)
-		(property "Datasheet" "~"
-			(at 34.29 106.68 0)
-			(effects
-				(font
-					(size 1.27 1.27)
-				)
-				(hide yes)
-			)
-		)
-		(property "Description" "Resistor, US symbol"
-			(at 34.29 106.68 0)
-			(effects
-				(font
-					(size 1.27 1.27)
-				)
-				(hide yes)
-			)
-		)
-		(pin "1"
-		)
-		(pin "2"
-		)
-		(instances
-			(project ""
-				(path "/da3163b4-b098-4cd4-9588-703f26f78e93"
-					(reference "R1")
-					(unit 1)
-				)
