File: Supplemental/SFX-Breakout/KiCad/SFX-BO-01/SFX-BO-01.kicad_sch (KiCad schematic)
At the start: 36 parts, among them J1 TB111-2-3-U-1-1, J10 Faston #250, J11 ATX/SFX 24pin, J12 Faston #250, J13 Faston #250, J14 Faston #250, J15 Faston #250, J16 Faston #250, J17 Faston #250, J18 XH-3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

Commit message: [SFX-BO-01] Snapshot to 1st PCB build
Parts:
- J1, J2, J3, J4: footprint (none) -> 01_Local_FP:TerminalBlock_Alphaplus_TB111-2-3-U-1-1_1x03_P5.08mm_Horizontal
- J10, J12, J13, J14, J15, J16, J17, J5, J6, J7, J8, J9: footprint (none) -> 01_Local_FP:Faston_PC250
- R1, R5, R6: footprint (none) -> 01_Local_FP:R_Axial_DIN0207_L6.3mm_D2.5mm_P15.24mm_Horizontal_TOSA
- R10, R2, R3, R4, R7, R8, R9: footprint (none) -> 01_Local_FP:R_Axial_DIN0207_L6.3mm_D2.5mm_P2.54mm_Vertical_TOSA
- SW1: footprint (none) -> 01_Local_FP:SW_Push_2P2T_Toggle_PB-22E85L
Connections:
- net PS_ON is gone; now on net PS_ON#: R6.2
- net +12V: now also J2.1 (Pin_1), J4.3 (Pin_3); no longer J2.3 (Pin_3), J4.1 (Pin_1)
- net +3.3V: now also J1.3 (Pin_3), J3.1 (Pin_1); no longer J1.1 (Pin_1), J11.12 (Pin_12), J3.3 (Pin_3)
- net +5V: now also J1.1 (Pin_1), J4.1 (Pin_1); no longer J1.3 (Pin_3), J4.3 (Pin_3)
- net +5VSB: now also J2.3 (Pin_3); no longer J2.1 (Pin_1)
- net -12V: now also J3.3 (Pin_3); no longer J3.1 (Pin_1)
- no-connect marks 3 -> 4
Other:
- moved on the sheet: J3, J4
Changed lines of the file:
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@@
 	(title_block
 		(title "SFX Breakout board （EvbPusher project)")
-		(date "2025-11-22")
+		(date "2026-02-26")
 		(rev "0.1.0")
 		(company "田中屋電脳部")
@@
 	)
 	(junction
-		(at 105.41 161.29)
-		(diameter 0)
-		(color 0 0 0 0)
-	)
-	(junction
 		(at 67.31 123.19)
 		(diameter 0)
@@
 	)
 	(no_connect
+		(at 92.71 186.69)
+	)
+	(no_connect
 		(at 80.01 176.53)
 	)
@@
 	(wire
 		(pts
-			(xy 105.41 186.69) (xy 105.41 161.29)
-		)
-		(stroke
-			(width 0)
-			(type default)
-		)
-	)
-	(wire
-		(pts
 			(xy 111.76 166.37) (xy 111.76 156.21)
 		)
@@
 	(wire
 		(pts
-			(xy 92.71 186.69) (xy 105.41 186.69)
-		)
-		(stroke
-			(width 0)
-			(type default)
-		)
-	)
-	(wire
-		(pts
 			(xy 96.52 163.83) (xy 96.52 168.91)
 		)
@@
 		)
 	)
-	(label "PS_ON"
+	(label "PS_ON#"
 		(at 189.23 41.91 180)
 		(effects
@@
 			)
 		)
-		(property "Footprint" ""
+		(property "Footprint" "01_Local_FP:R_Axial_DIN0207_L6.3mm_D2.5mm_P15.24mm_Horizontal_TOSA"
 			(at 170.434 40.894 90)
 			(effects
@@
 			)
 		)
-		(property "Footprint" ""
+		(property "Footprint" "01_Local_FP:Faston_PC250"
 			(at 59.69 102.87 0)
 			(effects
@@
 			)
 		)
-		(property "Footprint" ""
+		(property "Footprint" "01_Local_FP:Faston_PC250"
 			(at 100.33 106.68 0)
 			(effects
@@
 			)
 		)
-		(property "Footprint" ""
+		(property "Footprint" "01_Local_FP:R_Axial_DIN0207_L6.3mm_D2.5mm_P2.54mm_Vertical_TOSA"
 			(at 181.864 90.424 90)
 			(effects
@@
 			)
 		)
-		(property "Footprint" ""
+		(property "Footprint" "01_Local_FP:Faston_PC250"
 			(at 100.33 119.38 0)
 			(effects
@@
 			)
 		)
-		(property "Footprint" ""
+		(property "Footprint" "01_Local_FP:Faston_PC250"
 			(at 59.69 127 0)
 			(effects
@@
 			)
 		)
-		(property "Footprint" ""
+		(property "Footprint" "01_Local_FP:SW_Push_2P2T_Toggle_PB-22E85L"
 			(at 147.32 39.37 0)
 			(effects
@@
 			)
 		)
-		(property "Footprint" ""
+		(property "Footprint" "01_Local_FP:Faston_PC250"
 			(at 59.69 110.49 0)
 			(effects
@@
 			)
 		)
-		(property "Footprint" ""
+		(property "Footprint" "01_Local_FP:Faston_PC250"
 			(at 59.69 106.68 0)
 			(effects
@@
 			)
 		)
-		(property "Footprint" ""
+		(property "Footprint" "01_Local_FP:R_Axial_DIN0207_L6.3mm_D2.5mm_P2.54mm_Vertical_TOSA"
 			(at 205.994 110.236 90)
 			(effects
@@
 			)
 		)
-		(property "Footprint" ""
+		(property "Footprint" "01_Local_FP:R_Axial_DIN0207_L6.3mm_D2.5mm_P2.54mm_Vertical_TOSA"
 			(at 219.964 51.054 90)
 			(effects
@@
 			)
 		)
-		(property "Footprint" ""
+		(property "Footprint" "01_Local_FP:R_Axial_DIN0207_L6.3mm_D2.5mm_P2.54mm_Vertical_TOSA"
 			(at 219.964 61.214 90)
 			(effects
@@
 			)
 		)
-		(property "Footprint" ""
+		(property "Footprint" "01_Local_FP:Faston_PC250"
 			(at 100.33 123.19 0)
 			(effects
@@
 	(symbol
 		(lib_id "Connector:Screw_Terminal_01x03")
-		(at 59.69 49.53 180)
+		(at 59.69 49.53 0)
+		(mirror y)
 		(unit 1)
 		(exclude_from_sim no)
@@
 		(dnp no)
 		(property "Reference" "J3"
-			(at 59.436 42.418 0)
+			(at 59.436 56.642 0)
 			(effects
 				(font
@@
 		)
 		(property "Value" "TB111-2-3-U-1-1"
-			(at 50.8 44.45 0)
+			(at 50.8 54.61 0)
 			(effects
 				(font
@@
 			)
 		)
-		(property "Footprint" ""
+		(property "Footprint" "01_Local_FP:TerminalBlock_Alphaplus_TB111-2-3-U-1-1_1x03_P5.08mm_Horizontal"
 			(at 59.69 49.53 0)
 			(effects
@@
 		(lib_id "Connector:Screw_Terminal_01x03")
 		(at 100.33 49.53 0)
+		(mirror x)
 		(unit 1)
 		(exclude_from_sim no)
@@
 		(dnp no)
 		(property "Reference" "J1"
-			(at 99.06 41.402 0)
+			(at 99.06 57.658 0)
 			(effects
 				(font
@@
 		)
 		(property "Value" "TB111-2-3-U-1-1"
-			(at 99.314 43.688 0)
+			(at 99.314 55.372 0)
 			(effects
 				(font
@@
 			)
 		)
-		(property "Footprint" ""
+		(property "Footprint" "01_Local_FP:TerminalBlock_Alphaplus_TB111-2-3-U-1-1_1x03_P5.08mm_Horizontal"
 			(at 100.33 49.53 0)
 			(effects
@@
 			)
 		)
-		(property "Footprint" ""
+		(property "Footprint" "01_Local_FP:R_Axial_DIN0207_L6.3mm_D2.5mm_P2.54mm_Vertical_TOSA"
 			(at 219.964 71.374 90)
 			(effects
@@
 		(lib_id "Connector:Screw_Terminal_01x03")
 		(at 100.33 66.04 0)
+		(mirror x)
 		(unit 1)
 		(exclude_from_sim no)
@@
 		(dnp no)
 		(property "Reference" "J2"
-			(at 99.06 58.166 0)
+			(at 99.06 73.914 0)
 			(effects
 				(font
@@
 		)
 		(property "Value" "TB111-2-3-U-1-1"
-			(at 99.568 60.198 0)
+			(at 99.568 71.882 0)
 			(effects
 				(font
@@
 			)
 		)
-		(property "Footprint" ""
+		(property "Footprint" "01_Local_FP:TerminalBlock_Alphaplus_TB111-2-3-U-1-1_1x03_P5.08mm_Horizontal"
 			(at 100.33 66.04 0)
 			(effects
@@
 			)
 		)
-		(property "Footprint" ""
+		(property "Footprint" "01_Local_FP:R_Axial_DIN0207_L6.3mm_D2.5mm_P2.54mm_Vertical_TOSA"
 			(at 181.864 115.824 90)
 			(effects
@@
 			)
 		)
-		(property "Footprint" ""
+		(property "Footprint" "01_Local_FP:R_Axial_DIN0207_L6.3mm_D2.5mm_P2.54mm_Vertical_TOSA"
 			(at 181.864 103.124 90)
 			(effects
@@
 			)
 		)
-		(property "Footprint" ""
+		(property "Footprint" "01_Local_FP:R_Axial_DIN0207_L6.3mm_D2.5mm_P15.24mm_Horizontal_TOSA"
 			(at 147.574 90.424 90)
 			(effects
@@
 			)
 		)
-		(property "Footprint" ""
+		(property "Footprint" "01_Local_FP:Faston_PC250"
 			(at 100.33 102.87 0)
 			(effects
@@
 			)
 		)
-		(property "Footprint" ""
+		(property "Footprint" "01_Local_FP:R_Axial_DIN0207_L6.3mm_D2.5mm_P15.24mm_Horizontal_TOSA"
 			(at 188.214 155.194 90)
 			(effects
@@
 			)
 		)
-		(property "Footprint" ""
+		(property "Footprint" "01_Local_FP:Faston_PC250"
 			(at 100.33 127 0)
 			(effects
@@
 	(symbol
 		(lib_id "Connector:Screw_Terminal_01x03")
-		(at 59.69 66.04 180)
+		(at 59.69 66.04 0)
+		(mirror y)
 		(unit 1)
 		(exclude_from_sim no)
@@
 		(dnp no)
 		(property "Reference" "J4"
-			(at 59.436 58.674 0)
+			(at 59.436 73.406 0)
 			(effects
 				(font
@@
 		)
 		(property "Value" "TB111-2-3-U-1-1"
-			(at 60.706 60.96 0)
+			(at 60.706 71.12 0)
 			(effects
 				(font
@@
 			)
 		)
-		(property "Footprint" ""
+		(property "Footprint" "01_Local_FP:TerminalBlock_Alphaplus_TB111-2-3-U-1-1_1x03_P5.08mm_Horizontal"
 			(at 59.69 66.04 0)
 			(effects
@@
 			)
 		)
-		(property "Footprint" ""
+		(property "Footprint" "01_Local_FP:Faston_PC250"
 			(at 100.33 110.49 0)
 			(effects
@@
 			)
 		)
-		(property "Footprint" ""
+		(property "Footprint" "01_Local_FP:Faston_PC250"
 			(at 59.69 119.38 0)
 			(effects
@@
 			)
 		)
-		(property "Footprint" ""
+		(property "Footprint" "01_Local_FP:Faston_PC250"
 			(at 59.69 123.19 0)
 			(effects
